Commit message: Renamed arm_urdf3 to arm_urdf

File: src/arm_urdf/urdf/rover_urdf3.urdf (robot description, URDF)
Before this commit: robot arm_urdf3, 7 links, 6 joints
Links:
- link Link_1: geometry collision mesh filename=package://arm_urdf/meshes/collision/Link_1.STL; visual mesh filename=package://arm_urdf/meshes/visual/Link_1.STL
- link Link_2: geometry collision mesh filename=package://arm_urdf/meshes/collision/Link_2.STL; visual mesh filename=package://arm_urdf/meshes/visual/Link_2.STL
- link Link_3: geometry collision mesh filename=package://arm_urdf/meshes/collision/Link_3.STL; visual mesh filename=package://arm_urdf/meshes/visual/Link_3.STL
- link Link_4: geometry collision mesh filename=package://arm_urdf/meshes/collision/Link_4.STL; visual mesh filename=package://arm_urdf/meshes/visual/Link_4.STL
- link Link_5: geometry collision mesh filename=package://arm_urdf/meshes/collision/Link_5.STL; visual mesh filename=package://arm_urdf/meshes/visual/Link_5.STL
- link Link_6: geometry collision mesh filename=package://arm_urdf/meshes/collision/Link_6.STL; visual mesh filename=package://arm_urdf/meshes/visual/Link_6.STL
- link Link_7: geometry collision mesh filename=package://arm_urdf/meshes/collision/Link_7.STL; visual mesh filename=package://arm_urdf/meshes/visual/Link_7.STL
