Commit message: WIP

File: src/arm_urdf/urdf/arm_urdf.urdf (robot description, URDF)
Before this commit: robot arm_urdf, 9 links, 8 joints
Joints:
- joint Joint_1: limit lower=-1.50 upper=4.0 effort=100.0 velocity=0.5 -> lower=-3.1 upper=1.7 effort=100.0 velocity=0.5

Commit message: Don't ask me

File: src/arm_urdf/urdf/arm_urdf.urdf (robot description, URDF)
Before this commit: robot arm_urdf, 7 links, 6 joints
Joints:
- joint Joint_4: limit lower=-3.14 upper=3.14 effort=100.0 velocity=0.03688 -> lower=-3.14 upper=3.14 effort=100.0 velocity=0.60385
- joint Joint_5: limit lower=-2.0944 upper=1.0472 effort=100.0 velocity=1.0 -> lower=-2.0944 upper=1.0472 effort=100.0 velocity=0.0415
- joint Joint_6: limit lower=-3.14 upper=3.14 effort=100.0 velocity=1.0 -> lower=-3.14 upper=3.14 effort=100.0 velocity=0.28545

Commit message: Technically works

File: src/arm_urdf/urdf/arm_urdf.urdf (robot description, URDF)
Before this commit: robot arm_urdf, 7 links, 6 joints
Joints:
- joint Joint_5: limit lower=-2.0944 upper=1.0472 effort=100.0 velocity=1.0 -> lower=-2.0944 upper=1.0472 effort=100.0 velocity=0.0202
- joint Joint_6: limit lower=-3.14 upper=3.14 effort=100.0 velocity=1.0 -> lower=-3.14 upper=3.14 effort=100.0 velocity=0.28545

Commit message: arm tuning and controls adjustment

File: src/arm_urdf/urdf/arm_urdf.urdf (robot description, URDF)
Before this commit: robot arm_urdf, 9 links, 8 joints
Joints:
- joint Joint_1: limit lower=-1.57 upper=1.57 effort=100.0 velocity=1.0 -> lower=-100.0 upper=100.0 effort=100.0 velocity=1.0
- joint Joint_2: limit lower=-0.488692 upper=0.279253 effort=100.0 velocity=0.08 -> lower=-1.2885438618239387 upper=-0.38196121618352463 effort=100.0 velocity=0.10
- joint Joint_3: limit lower=-1.2 upper=0.15 effort=100.0 velocity=0.08 -> lower=-0.9273642258919734 upper=0.0 effort=100.0 velocity=0.08
- joint Joint_4: limit lower=-3.14 upper=3.14 effort=100.0 velocity=1.0 -> lower=-30.14 upper=30.14 effort=100.0 velocity=1.0
- joint Joint_5: limit lower=-2.0944 upper=1.0472 effort=100.0 velocity=1.0 -> lower=0.0 upper=2.4344275103745123 effort=100.0 velocity=1.0

Commit message: get arm working again

File: src/arm_urdf/urdf/arm_urdf.urdf (robot description, URDF)
Before this commit: robot arm_urdf, 9 links, 8 joints
Joints:
- joint Joint_2: limit lower=-1.2885438618239387 upper=-0.38196121618352463 effort=100.0 velocity=0.10 -> lower=-0.65 upper=0.2361743685324814 effort=100.0 velocity=0.10
- joint Joint_3: limit lower=-0.9273642258919734 upper=0.0 effort=100.0 velocity=0.08 -> lower=-0.7417525505578109 upper=0.2139174802949436 effort=100.0 velocity=0.08
- joint Joint_5: limit lower=0.0 upper=2.4344275103745123 effort=100.0 velocity=1.0 -> lower=-1.6805630104816343 upper=0.8274955777113892 effort=100.0 velocity=1.0

Commit message: limits and offsets set better

File: src/arm_urdf/urdf/arm_urdf.urdf (robot description, URDF)
Before this commit: robot arm_urdf, 9 links, 8 joints
Joints:
- joint Joint_1: limit lower=-100.0 upper=100.0 effort=100.0 velocity=1.0 -> lower=-3.981728005722112 upper=-1.1116499515880771 effort=100.0 velocity=1.0
- joint Joint_5: limit lower=-1.6805630104816343 upper=0.8274955777113892 effort=100.0 velocity=1.0 -> lower=-1.599417185 upper=1.1678841562 effort=100.0 velocity=1.0

Commit message: cutting it close arn't ya!

File: src/arm_urdf/urdf/arm_urdf.urdf (robot description, URDF)
Before this commit: robot arm_urdf, 9 links, 8 joints
Joints:
- joint Joint_1: limit lower=-3.981728005722112 upper=-1.1116499515880771 effort=100.0 velocity=1.0 -> lower=-100.0 upper=100.0 effort=100.0 velocity=1.0

Commit message: s

File: src/arm_urdf/urdf/arm_urdf.urdf (robot description, URDF)
Before this commit: robot arm_urdf, 9 links, 8 joints
Joints:
- joint Joint_1: limit lower=-3.14 upper=3.14 effort=100.0 velocity=0.5 -> lower=-1.50 upper=4.0 effort=100.0 velocity=0.5

Commit message: arm_tuning changes

File: src/arm_urdf/urdf/arm_urdf.urdf (robot description, URDF)
Before this commit: robot arm_urdf, 9 links, 8 joints
Joints:
- joint Joint_1: limit lower=-3.14 upper=3.14 effort=100.0 velocity=0.5 -> lower=-3.1 upper=1.7 effort=100.0 velocity=0.5
