Commit message: Joint limits added

File: src/arm_urdf3/urdf/arm_urdf3.urdf (robot description, URDF)
Before this commit: robot arm_urdf3, 7 links, 6 joints
Joints:
- joint Joint_1: limit (none) -> lower=-1.57 upper=1.57 effort=100.0 velocity=1.0; type continuous -> revolute
- joint Joint_2: limit (none) -> lower=-0.3858 upper=0.4626 effort=100.0 velocity=0.0234; type continuous -> revolute
- joint Joint_3: limit (none) -> lower=-0.6578 upper=0.3033 effort=100.0 velocity=0.03688; type continuous -> revolute
- joint Joint_4: limit (none) -> lower=-3.14 upper=3.14 effort=100.0 velocity=0.03688; type continuous -> revolute
- joint Joint_5: limit (none) -> lower=-2.0944 upper=1.0472 effort=100.0 velocity=1.0; type continuous -> revolute
- joint Joint_6: limit (none) -> lower=-3.14 upper=3.14 effort=100.0 velocity=1.0; type continuous -> revolute
