Commit message: Apply suggestions from code review
Co-authored-by: ConnorNeed <129120300+ConnorNeed@users.noreply.github.com>

File: src/arm_srdf3/config/arm_urdf3.ros2_control.xacro (robot description, xacro)
@@ -1,5 +1,5 @@
 <?xml version="1.0"?>
 <robot xmlns:xacro="http://www.ros.org/wiki/xacro">
-    <xacro:macro name="arm_urdf3_ros2_control" params="name initial_positions_file">
+    <xacro:macro name="arm_urdf_ros2_control" params="name initial_positions_file">
         <xacro:property name="initial_positions" value="${load_yaml(initial_positions_file)['initial_positions']}"/>
         <ros2_control name="${name}" type="system">

File: src/arm_srdf3/config/arm_urdf3.urdf.xacro (robot description, xacro)
@@ -1,7 +1,7 @@
 <?xml version="1.0"?>
-<robot xmlns:xacro="http://www.ros.org/wiki/xacro" name="arm_urdf3">
+<robot xmlns:xacro="http://www.ros.org/wiki/xacro" name="arm_urdf">
     <xacro:arg name="initial_positions_file" default="initial_positions.yaml" />
     <!-- Import arm_urdf3 urdf file -->
-    <xacro:include filename="$(find arm_urdf3)/urdf/arm_urdf3.urdf" />
+    <xacro:include filename="$(find arm_urdf)/urdf/arm_urdf.urdf" />
     <!-- Import control_xacro -->
     <xacro:include filename="arm_urdf3.ros2_control.xacro" />
