Commit message: Renamed folders

File: src/arm_srdf/config/arm_urdf.urdf.xacro (robot description, xacro)
@@ -2,8 +2,8 @@
 <robot xmlns:xacro="http://www.ros.org/wiki/xacro" name="arm_urdf">
     <xacro:arg name="initial_positions_file" default="initial_positions.yaml" />
-    <!-- Import arm_urdf3 urdf file -->
+    <!-- Import arm_urdf urdf file -->
     <xacro:include filename="$(find arm_urdf)/urdf/arm_urdf.urdf" />
     <!-- Import control_xacro -->
-    <xacro:include filename="arm_urdf3.ros2_control.xacro" />
-    <xacro:arm_urdf3_ros2_control name="FakeSystem" initial_positions_file="$(arg initial_positions_file)"/>
+    <xacro:include filename="arm_urdf.ros2_control.xacro" />
+    <xacro:arm_urdf_ros2_control name="FakeSystem" initial_positions_file="$(arg initial_positions_file)"/>
 </robot>

File: src/arm_urdf/urdf/arm_urdf.urdf (robot description, URDF)
Before this commit: robot arm_urdf3, 7 links, 6 joints
Links:
- link Link_1: geometry collision mesh filename=package://arm_urdf/meshes/visual/Link_1.STL; visual mesh filename=package://arm_urdf/meshes/visual/Link_1.STL
- link Link_2: geometry collision mesh filename=package://arm_urdf/meshes/visual/Link_2.STL; visual mesh filename=package://arm_urdf/meshes/visual/Link_2.STL
- link Link_3: geometry collision mesh filename=package://arm_urdf/meshes/visual/Link_3.STL; visual mesh filename=package://arm_urdf/meshes/visual/Link_3.STL
- link Link_4: geometry collision mesh filename=package://arm_urdf/meshes/visual/Link_4.STL; visual mesh filename=package://arm_urdf/meshes/visual/Link_4.STL
- link Link_5: geometry collision mesh filename=package://arm_urdf/meshes/visual/Link_5.STL; visual mesh filename=package://arm_urdf/meshes/visual/Link_5.STL
- link Link_6: geometry collision mesh filename=package://arm_urdf/meshes/visual/Link_6.STL; visual mesh filename=package://arm_urdf/meshes/visual/Link_6.STL
- link Link_7: geometry collision mesh filename=package://arm_urdf/meshes/visual/Link_7.STL; visual mesh filename=package://arm_urdf/meshes/visual/Link_7.STL
