Commit message: Reformatted files

File: src/arm_srdf/config/arm_urdf.ros2_control.xacro (robot description, xacro)
@@ -6,9 +6,9 @@
             <hardware>
                 <!-- By default, set up controllers for simulation. This won't work on real hardware -->
-                <!--<plugin>mock_components/GenericSystem</plugin>-->
-                <plugin>ros2_control_rover_arm/RoverArmHardwareInterface</plugin>
+                <plugin>mock_components/GenericSystem</plugin>
             </hardware>
             <joint name="Joint_1">
                 <command_interface name="position"/>
+                <command_interface name="velocity"/>
                 <state_interface name="position">
                   <param name="initial_value">${initial_positions['Joint_1']}</param>
@@ -18,4 +18,5 @@
             <joint name="Joint_2">
                 <command_interface name="position"/>
+                <command_interface name="velocity"/>
                 <state_interface name="position">
                   <param name="initial_value">${initial_positions['Joint_2']}</param>
@@ -25,4 +26,5 @@
             <joint name="Joint_3">
                 <command_interface name="position"/>
+                <command_interface name="velocity"/>
                 <state_interface name="position">
                   <param name="initial_value">${initial_positions['Joint_3']}</param>
@@ -32,4 +34,5 @@
             <joint name="Joint_4">
                 <command_interface name="position"/>
+                <command_interface name="velocity"/>
                 <state_interface name="position">
                   <param name="initial_value">${initial_positions['Joint_4']}</param>
@@ -39,4 +42,5 @@
             <joint name="Joint_5">
                 <command_interface name="position"/>
+                <command_interface name="velocity"/>
                 <state_interface name="position">
                   <param name="initial_value">${initial_positions['Joint_5']}</param>
@@ -46,4 +50,5 @@
             <joint name="Joint_6">
                 <command_interface name="position"/>
+                <command_interface name="velocity"/>
                 <state_interface name="position">
                   <param name="initial_value">${initial_positions['Joint_6']}</param>

File: src/arm_urdf/urdf/arm_urdf.urdf (robot description, URDF)
Before this commit: robot arm_urdf, 7 links, 6 joints
Links:
- link Link_1: mass 3.331 -> 1.1012
- link Link_2: mass 0.51625 -> 0.73837
- link Link_3: mass 1.9352 -> 2.2244
- link Link_4: mass 0.90456 -> 0.72553
- link Link_5: mass 1.42 -> 0.90226
- link Link_6: mass 0.4426 -> 0.496128874632715
Joints:
- joint Joint_1: limit lower=-1.57 upper=1.57 effort=100.0 velocity=1.0 -> (none); origin xyz=0 0 0.0207625000000001 rpy=0 0 0 -> xyz=0 0 0.022287 rpy=0 0 0; type revolute -> continuous
- joint Joint_2: limit lower=-0.3858 upper=0.4626 effort=100.0 velocity=0.0234 -> (none); origin xyz=0 0 0.1 rpy=0 0 0 -> xyz=-0.03175 0 0.1 rpy=0 0 0; type revolute -> continuous
- joint Joint_3: limit lower=-0.6578 upper=0.3033 effort=100.0 velocity=0.03688 -> (none); origin xyz=0.558012701892218 0 0.466506350946108 rpy=0 0 0 -> xyz=0.4507 0 0.5371 rpy=0 0 0; type revolute -> continuous
- joint Joint_4: axis -0.866025403784437 0 0.500000000000002 -> -0.99059 0 0.1369; limit lower=-3.14 upper=3.14 effort=100.0 velocity=0.03688 -> (none); origin xyz=-0.0209336725054375 -0.000155363339502348 0.0120860614561421 rpy=0 0 0 -> xyz=0.03191 0 -0.0044098 rpy=0 0 0; type revolute -> continuous
- joint Joint_5: limit lower=-2.0944 upper=1.0472 effort=100.0 velocity=1.0 -> (none); origin xyz=0.63745932252309 0 -0.368037311456142 rpy=0 0 0 -> xyz=0.68151 0 -0.094183 rpy=0 0 0; type revolute -> continuous
- joint Joint_6: limit lower=-3.14 upper=3.14 effort=100.0 velocity=1.0 -> (none); origin xyz=0.0621500000000025 -0.0285875000000056 0 rpy=0 0 0 -> xyz=0.071675 -0.02785 0 rpy=0 0 0; type revolute -> continuous

Commit message: Added joint limits and a few other things

File: src/arm_srdf/config/arm_urdf.ros2_control.xacro (robot description, xacro)
@@ -6,5 +6,6 @@
             <hardware>
                 <!-- By default, set up controllers for simulation. This won't work on real hardware -->
-                <plugin>mock_components/GenericSystem</plugin>
+                <!--<plugin>mock_components/GenericSystem</plugin> !-->
+                <plugin>ros2_control_rover_arm/RoverArmHardwareInterface</plugin>
             </hardware>
             <joint name="Joint_1">

File: src/arm_urdf/urdf/arm_urdf.urdf (robot description, URDF)
Before this commit: robot arm_urdf, 7 links, 6 joints
Joints:
- joint Joint_2: limit lower=-0.3858 upper=0.4626 effort=100.0 velocity=0.0234 -> lower=-0.55 upper=0.3236 effort=100.0 velocity=0.0234
- joint Joint_3: limit lower=-0.6578 upper=0.3033 effort=100.0 velocity=0.03688 -> lower=-0.9032 upper=0.054 effort=100.0 velocity=0.03688

Commit message: New urdf (#66)
* Reformatted files

* Updated joint limits

* Added joint limits and a few other things

* Removed test-only file

* Update src/hardware/src/rover_arm.cpp

Co-authored-by: Connor Needham <129120300+ConnorNeed@users.noreply.github.com>

* Formatted

---------

Co-authored-by: Connor Needham <129120300+ConnorNeed@users.noreply.github.com>

File: src/arm_srdf/config/arm_urdf.ros2_control.xacro (robot description, xacro)
@@ -6,9 +6,10 @@
             <hardware>
                 <!-- By default, set up controllers for simulation. This won't work on real hardware -->
-                <!--<plugin>mock_components/GenericSystem</plugin>-->
+                <!--<plugin>mock_components/GenericSystem</plugin> !-->
                 <plugin>ros2_control_rover_arm/RoverArmHardwareInterface</plugin>
             </hardware>
             <joint name="Joint_1">
                 <command_interface name="position"/>
+                <command_interface name="velocity"/>
                 <state_interface name="position">
                   <param name="initial_value">${initial_positions['Joint_1']}</param>
@@ -18,4 +19,5 @@
             <joint name="Joint_2">
                 <command_interface name="position"/>
+                <command_interface name="velocity"/>
                 <state_interface name="position">
                   <param name="initial_value">${initial_positions['Joint_2']}</param>
@@ -25,4 +27,5 @@
             <joint name="Joint_3">
                 <command_interface name="position"/>
+                <command_interface name="velocity"/>
                 <state_interface name="position">
                   <param name="initial_value">${initial_positions['Joint_3']}</param>
@@ -32,4 +35,5 @@
             <joint name="Joint_4">
                 <command_interface name="position"/>
+                <command_interface name="velocity"/>
                 <state_interface name="position">
                   <param name="initial_value">${initial_positions['Joint_4']}</param>
@@ -39,4 +43,5 @@
             <joint name="Joint_5">
                 <command_interface name="position"/>
+                <command_interface name="velocity"/>
                 <state_interface name="position">
                   <param name="initial_value">${initial_positions['Joint_5']}</param>
@@ -46,4 +51,5 @@
             <joint name="Joint_6">
                 <command_interface name="position"/>
+                <command_interface name="velocity"/>
                 <state_interface name="position">
                   <param name="initial_value">${initial_positions['Joint_6']}</param>

File: src/arm_urdf/urdf/arm_urdf.urdf (robot description, URDF)
Before this commit: robot arm_urdf, 7 links, 6 joints
Links:
- link Link_1: mass 3.331 -> 1.1012
- link Link_2: mass 0.51625 -> 0.73837
- link Link_3: mass 1.9352 -> 2.2244
- link Link_4: mass 0.90456 -> 0.72553
- link Link_5: mass 1.42 -> 0.90226
- link Link_6: mass 0.4426 -> 0.496128874632715
Joints:
- joint Joint_1: origin xyz=0 0 0.0207625000000001 rpy=0 0 0 -> xyz=0 0 0.022287 rpy=0 0 0
- joint Joint_2: limit lower=-0.3858 upper=0.4626 effort=100.0 velocity=0.0234 -> lower=-0.55 upper=0.3236 effort=100.0 velocity=0.0234; origin xyz=0 0 0.1 rpy=0 0 0 -> xyz=-0.03175 0 0.1 rpy=0 0 0
- joint Joint_3: limit lower=-0.6578 upper=0.3033 effort=100.0 velocity=0.03688 -> lower=-0.9032 upper=0.054 effort=100.0 velocity=0.03688; origin xyz=0.558012701892218 0 0.466506350946108 rpy=0 0 0 -> xyz=0.4507 0 0.5371 rpy=0 0 0
- joint Joint_4: axis -0.866025403784437 0 0.500000000000002 -> -0.99059 0 0.1369; origin xyz=-0.0209336725054375 -0.000155363339502348 0.0120860614561421 rpy=0 0 0 -> xyz=0.03191 0 -0.0044098 rpy=0 0 0
- joint Joint_5: origin xyz=0.63745932252309 0 -0.368037311456142 rpy=0 0 0 -> xyz=0.68151 0 -0.094183 rpy=0 0 0
- joint Joint_6: origin xyz=0.0621500000000025 -0.0285875000000056 0 rpy=0 0 0 -> xyz=0.071675 -0.02785 0 rpy=0 0 0

Commit message: Velocity Control IK

File: src/arm_srdf/config/arm_urdf.ros2_control.xacro (robot description, xacro)
@@ -1,61 +1,48 @@
 <?xml version="1.0"?>
 <robot xmlns:xacro="http://www.ros.org/wiki/xacro">
-    <xacro:macro name="arm_urdf_ros2_control" params="name initial_positions_file">
-        <xacro:property name="initial_positions" value="${load_yaml(initial_positions_file)['initial_positions']}"/>
-        <ros2_control name="${name}" type="system">
-            <hardware>
-                <!-- By default, set up controllers for simulation. This won't work on real hardware -->
-                <!--<plugin>mock_components/GenericSystem</plugin> !-->
-                <plugin>ros2_control_rover_arm/RoverArmHardwareInterface</plugin>
-            </hardware>
-            <joint name="Joint_1">
-                <command_interface name="position"/>
-                <command_interface name="velocity"/>
-                <state_interface name="position">
-                  <param name="initial_value">${initial_positions['Joint_1']}</param>
-                </state_interface>
-                <state_interface name="velocity"/>
-            </joint>
-            <joint name="Joint_2">
-                <command_interface name="position"/>
-                <command_interface name="velocity"/>
-                <state_interface name="position">
-                  <param name="initial_value">${initial_positions['Joint_2']}</param>
-                </state_interface>
-                <state_interface name="velocity"/>
-            </joint>
-            <joint name="Joint_3">
-                <command_interface name="position"/>
-                <command_interface name="velocity"/>
-                <state_interface name="position">
-                  <param name="initial_value">${initial_positions['Joint_3']}</param>
-                </state_interface>
-                <state_interface name="velocity"/>
-            </joint>
-            <joint name="Joint_4">
-                <command_interface name="position"/>
-                <command_interface name="velocity"/>
-                <state_interface name="position">
-                  <param name="initial_value">${initial_positions['Joint_4']}</param>
-                </state_interface>
-                <state_interface name="velocity"/>
-            </joint>
-            <joint name="Joint_5">
-                <command_interface name="position"/>
-                <command_interface name="velocity"/>
-                <state_interface name="position">
-                  <param name="initial_value">${initial_positions['Joint_5']}</param>
-                </state_interface>
-                <state_interface name="velocity"/>
-            </joint>
-            <joint name="Joint_6">
-                <command_interface name="position"/>
-                <command_interface name="velocity"/>
-                <state_interface name="position">
-                  <param name="initial_value">${initial_positions['Joint_6']}</param>
-                </state_interface>
-                <state_interface name="velocity"/>
-            </joint>
-        </ros2_control>
-    </xacro:macro>
+  <xacro:macro name="arm_urdf_ros2_control" params="name">
+    <ros2_control name="${name}" type="system">
+      <hardware>
+        <!-- By default, set up controllers for simulation. This won't work on real hardware -->
+        <!--<plugin>mock_components/GenericSystem</plugin> !-->
+        <plugin>ros2_control_rover_arm/RoverArmHardwareInterface</plugin>
+      </hardware>
+      <joint name="Joint_1">
+        <param name="node_name">base</param>
+        <command_interface name="velocity"/>
+        <state_interface name="position"/>
+        <state_interface name="velocity"/>
+      </joint>
+      <joint name="Joint_2">
+        <param name="node_name">act1</param>
+        <command_interface name="velocity"/>
+        <state_interface name="position"/>
+        <state_interface name="velocity"/>
+      </joint>
+      <joint name="Joint_3">
+        <param name="node_name">act2</param>
+        <command_interface name="velocity"/>
+        <state_interface name="position"/>
+        <state_interface name="velocity"/>
+      </joint>
+      <joint name="Joint_4">
+        <param name="node_name">elbow</param>
+        <command_interface name="velocity"/>
+        <state_interface name="position"/>
+        <state_interface name="velocity"/>
+      </joint>
+      <joint name="Joint_5">
+        <param name="node_name">wristTilt</param>
+        <command_interface name="velocity"/>
+        <state_interface name="position"/>
+        <state_interface name="velocity"/>
+      </joint>
+      <joint name="Joint_6">
+        <param name="node_name">wristTurn</param>
+        <command_interface name="velocity"/>
+        <state_interface name="position"/>
+        <state_interface name="velocity"/>
+      </joint>
+    </ros2_control>
+  </xacro:macro>
 </robot>

File: src/arm_srdf/config/arm_urdf.urdf.xacro (robot description, xacro)
@@ -1,9 +1,8 @@
 <?xml version="1.0"?>
 <robot xmlns:xacro="http://www.ros.org/wiki/xacro" name="arm_urdf">
-    <xacro:arg name="initial_positions_file" default="initial_positions.yaml" />
     <!-- Import arm_urdf urdf file -->
     <xacro:include filename="$(find arm_urdf)/urdf/arm_urdf.urdf" />
     <!-- Import control_xacro -->
     <xacro:include filename="arm_urdf.ros2_control.xacro" />
-    <xacro:arm_urdf_ros2_control name="FakeSystem" initial_positions_file="$(arg initial_positions_file)"/>
+    <xacro:arm_urdf_ros2_control name="ArmSystem"/>
 </robot>

File: src/arm_urdf/urdf/arm_urdf.urdf (robot description, URDF)
Before this commit: robot arm_urdf, 7 links, 6 joints
Links:
- added link arm_base_link
- added link eef_link
Joints:
- added joint arm_base_joint: type fixed, parent arm_base_link, child Link_1, origin xyz=0.0 0.0 0.0  rpy=0 0 0
- added joint eef_joint: type fixed, parent Link_7, child eef_link, origin xyz=0.2 0.0 0.0  rpy=0 0 0
- joint Joint_2: limit lower=-0.55 upper=0.3236 effort=100.0 velocity=0.0234 -> lower=-0.488692 upper=0.279253 effort=100.0 velocity=0.08
- joint Joint_3: limit lower=-0.9032 upper=0.054 effort=100.0 velocity=0.03688 -> lower=-1.2 upper=0.15 effort=100.0 velocity=0.08
- joint Joint_4: limit lower=-3.14 upper=3.14 effort=100.0 velocity=0.03688 -> lower=-3.14 upper=3.14 effort=100.0 velocity=1.0
- joint Joint_6: limit lower=-3.14 upper=3.14 effort=100.0 velocity=1.0 -> effort=100.0 velocity=1.5; type revolute -> continuous

Commit message: tune: needs more tuning but this is basically working

File: src/arm_srdf/config/arm_urdf.ros2_control.xacro (robot description, xacro)
@@ -9,13 +9,15 @@
       </hardware>
       <joint name="Joint_1">
-        <param name="can_id">1</param>
-        <param name="kP">0.1</param>
+        <param name="can_id">10</param>
+        <param name="kP">3.0</param>
         <param name="kI">0.0</param>
-        <param name="kD">0.0</param>
-        <param name="control_type">velocity</param> <!-- or "position" -->
+        <param name="kD">1.0</param>
+        <param name="kF">0.5</param>
         <param name="sensor_type">absolute</param> <!-- or "quadrature" -->
         <param name="sensor_ticks">4096</param>
         <param name="sensor_offset">0.0</param>
         <param name="crossover">true</param> <!-- or "continuous" -->
+        <param name="invert">false</param>
+        <param name="invert_sensor">true</param>
         <command_interface name="velocity"/>
         <state_interface name="position"/>
@@ -23,13 +25,15 @@
       </joint>
       <joint name="Joint_2">
-        <param name="can_id">2</param>
-        <param name="kP">0.1</param>
+        <param name="can_id">11</param>
+        <param name="kP">10.0</param>
         <param name="kI">0.0</param>
-        <param name="kD">0.0</param>
-        <param name="control_type">velocity</param> <!-- or "position" -->
+        <param name="kD">10.0</param>
+        <param name="kF">100</param>
         <param name="sensor_type">absolute</param> <!-- or "quadrature" -->
         <param name="sensor_ticks">4096</param>
-        <param name="sensor_offset">0.0</param>
+        <param name="sensor_offset">3.14</param>
         <param name="crossover">true</param> <!-- or "continuous" -->
+        <param name="invert">false</param>
+        <param name="invert_sensor">true</param>
         <command_interface name="velocity"/>
         <state_interface name="position"/>
@@ -37,13 +41,15 @@
       </joint>
       <joint name="Joint_3">
-        <param name="can_id">3</param>
-        <param name="kP">0.1</param>
+        <param name="can_id">14</param>
+        <param name="kP">30.0</param>
         <param name="kI">0.0</param>
-        <param name="kD">0.0</param>
-        <param name="control_type">velocity</param> <!-- or "position" -->
+        <param name="kD">3.0</param>
+        <param name="kF">125</param>
         <param name="sensor_type">absolute</param> <!-- or "quadrature" -->
         <param name="sensor_ticks">4096</param>
-        <param name="sensor_offset">0.0</param>
+        <param name="sensor_offset">2.02401481</param>
         <param name="crossover">true</param> <!-- or "continuous" -->
+        <param name="invert">true</param>
+        <param name="invert_sensor">false</param>
         <command_interface name="velocity"/>
         <state_interface name="position"/>
@@ -51,13 +57,15 @@
       </joint>
       <joint name="Joint_4">
-        <param name="can_id">4</param>
-        <param name="kP">0.1</param>
+        <param name="can_id">15</param>
+        <param name="kP">2.0</param>
         <param name="kI">0.0</param>
         <param name="kD">0.0</param>
-        <param name="control_type">velocity</param> <!-- or "position" -->
+        <param name="kF">5.0</param>
         <param name="sensor_type">absolute</param> <!-- or "quadrature" -->
         <param name="sensor_ticks">4096</param>
-        <param name="sensor_offset">0.0</param>
+        <param name="sensor_offset">4.54</param>
         <param name="crossover">true</param> <!-- or "continuous" -->
+        <param name="invert">false</param>
+        <param name="invert_sensor">false</param>
         <command_interface name="velocity"/>
         <state_interface name="position"/>
@@ -65,13 +73,15 @@
       </joint>
       <joint name="Joint_5">
-        <param name="can_id">5</param>
-        <param name="kP">0.1</param>
+        <param name="can_id">12</param>
+        <param name="kP">20.0</param>
         <param name="kI">0.0</param>
         <param name="kD">0.0</param>
-        <param name="control_type">velocity</param> <!-- or "position" -->
+        <param name="kF">7.8</param>
         <param name="sensor_type">absolute</param> <!-- or "quadrature" -->
         <param name="sensor_ticks">4096</param>
-        <param name="sensor_offset">0.0</param>
+        <param name="sensor_offset">2.54</param>
         <param name="crossover">true</param> <!-- or "continuous" -->
+        <param name="invert">true</param>
+        <param name="invert_sensor">true</param>
         <command_interface name="velocity"/>
         <state_interface name="position"/>
@@ -79,13 +89,15 @@
       </joint>
       <joint name="Joint_6">
-        <param name="can_id">6</param>
-        <param name="kP">0.1</param>
+        <param name="can_id">13</param>
+        <param name="kP">0.012</param>
         <param name="kI">0.0</param>
         <param name="kD">0.0</param>
-        <param name="control_type">velocity</param> <!-- or "position" -->
-        <param name="sensor_type">absolute</param> <!-- or "quadrature" -->
-        <param name="sensor_ticks">4096</param>
+        <param name="kF">0.005</param>
+        <param name="sensor_type">quadrature</param> <!-- or "quadrature" -->
+        <param name="sensor_ticks">1163000</param> <!-- TODO: this number is close but not quite -->
         <param name="sensor_offset">0.0</param>
         <param name="crossover">true</param> <!-- or "continuous" -->
+        <param name="invert">true</param>
+        <param name="invert_sensor">true</param>
         <command_interface name="velocity"/>
         <state_interface name="position"/>

File: src/arm_urdf/urdf/arm_urdf.urdf (robot description, URDF)
Before this commit: robot arm_urdf, 9 links, 8 joints
Joints:
- joint Joint_1: limit lower=-100.0 upper=100.0 effort=100.0 velocity=1.0 -> lower=-3.14 upper=3.14 effort=100.0 velocity=0.5
- joint Joint_4: limit lower=-30.14 upper=30.14 effort=100.0 velocity=1.0 -> lower=-3.14 upper=3.14 effort=100.0 velocity=0.5
- joint Joint_6: limit effort=100.0 velocity=1.5 -> effort=100.0 velocity=1.0

Commit message: GCXpo arm tunings

File: src/arm_srdf/config/arm_urdf.ros2_control.xacro (robot description, xacro)
@@ -28,5 +28,5 @@
         <param name="kP">10.0</param>
         <param name="kI">0.0</param>
-        <param name="kD">10.0</param>
+        <param name="kD">0.0</param>
         <param name="kF">100</param>
         <param name="sensor_type">absolute</param> <!-- or "quadrature" -->
@@ -42,8 +42,8 @@
       <joint name="Joint_3">
         <param name="can_id">14</param>
-        <param name="kP">30.0</param>
+        <param name="kP">10.0</param>
         <param name="kI">0.0</param>
-        <param name="kD">3.0</param>
-        <param name="kF">125</param>
+        <param name="kD">0.0</param>
+        <param name="kF">60.0</param>
         <param name="sensor_type">absolute</param> <!-- or "quadrature" -->
         <param name="sensor_ticks">4096</param>

File: src/arm_urdf/urdf/arm_urdf.urdf (robot description, URDF)
Before this commit: robot arm_urdf, 9 links, 8 joints
Joints:
- joint Joint_3: limit lower=-0.7417525505578109 upper=0.2139174802949436 effort=100.0 velocity=0.08 -> lower=-1000000.0 upper=10000000.0 effort=100.0 velocity=0.08
